Commit message: try to accelerate using gpu

File: src/bar_examples/krytn/robot_description/krytn.urdf.xacro (robot description, xacro)
@@ -1,42 +1,28 @@
 <?xml version='1.0' encoding='utf-8'?>
 <robot xmlns:xacro="http://www.ros.org/wiki/xacro" name="krytn" encoding='UTF-8'>
-  <!-- Import and add robot components -->
+  <!-- Import macro definitions -->
   <xacro:include filename="$(find magni_description)/urdf/magni.urdf.xacro" />
   <xacro:include filename="$(find sensors)/realsense_d435/realsense.urdf.xacro" />
+  <!-- CORRECTED INCLUDE PATH FOR LIDAR -->
   <xacro:include filename="$(find sensors)/lidar_2d/lidar_2d.urdf.xacro" />
+  <xacro:include filename="$(find krytn)/robot_description/krytn.gz.xacro" />
+  <!-- Instantiate the Magni base -->
+  <xacro:magni_robot_base_definition/>
+  <link name="base_footprint"/>
+  <joint name="base_footprint_to_base_link_joint" type="fixed">
+    <parent link="base_footprint"/>
+    <child link="base_link"/>
+    <origin xyz="0 0 ${0.1}" rpy="0 0 0"/>
+    <!-- Assumes Magni wheel_r is 0.1 -->
+  </joint>
+  <!-- Instantiate the sensors, attaching to 'base_link' (which comes from Magni) -->
   <xacro:realsense world_link_name="base_link">
-    <origin xyz="0 0 0.3" rpy="0 0 0" />
+    <origin xyz="0.15 0 0.25" rpy="0 0 0" />
   </xacro:realsense>
   <xacro:lidar_2d world_link_name="base_link">
-    <origin xyz="0 0 0.15" rpy="0 0 0" />
+    <origin xyz="0.20 0 0.15" rpy="0 0 0" />
   </xacro:lidar_2d>
-<!-- krytn_tray link-->
-  <link name="krytn_tray">
-    <visual>
-      <!--Krytn_tray_part/Body.-->
-      <origin rpy="0.0 -0.0 0.0" xyz="0.0 0.0 0.0"/>
-      <geometry>
-        <mesh filename="package://krytn_tray/meshes/krytn_tray_ex_Body.dae"/>
-      </geometry>
-    </visual>
-    <collision>
-      <!--Krytn_tray_part/Body.-->
-      <origin rpy="0.0 -0.0 0.0" xyz="0.0 0.0 0.0"/>
-      <geometry>
-        <mesh filename="package://krytn_tray/meshes/krytn_tray_ex_Body.dae"/>
-      </geometry>
-    </collision>
-    <xacro:box_inertial_with_origin x="0.400" y="0.280" z="0.220" mass="1.0">
-      <origin xyz="0.0 0.0 0.0" rpy="0 0 0" />
-    </xacro:box_inertial_with_origin>
-  </link>
-  <!-- tray_joint-->
- <joint name="krytn_joint" type="fixed">
-    <parent link="base_link"/>
-    <child link="krytn_tray"/>
-    <origin rpy="0.0 -0.0 0.0" xyz="0.052 0.0 0.264"/>
-  </joint>
-  <!-- Configure Control of Joints -->
-  <ros2_control name="Krytn" type="system">
+  <!-- ros2_control setup for Krytn (using Magni's joints) -->
+  <ros2_control name="KrytnControlSystem" type="system">
     <hardware>
       <plugin>gz_ros2_control/GazeboSimSystem</plugin>
@@ -49,5 +35,5 @@
       <state_interface name="position"/>
       <state_interface name="velocity"/>
-      <state_interface name="effort" />
+      <state_interface name="effort"/>
     </joint>
     <joint name="right_wheel_joint">
@@ -58,8 +44,7 @@
       <state_interface name="position"/>
       <state_interface name="velocity"/>
-      <state_interface name="effort" />
+      <state_interface name="effort"/>
     </joint>
   </ros2_control>
-  <!-- Setup Gazebo plugins -->
   <gazebo>
     <plugin filename="gz_ros2_control-system" name="gz_ros2_control::GazeboSimROS2ControlPlugin">
@@ -70,7 +55,4 @@
       <parameters>$(find krytn)/config/diffdrive_control.yaml</parameters>
     </plugin>
-    <plugin filename="gz-sim-sensors-system" name="gz::sim::systems::Sensors">
-      <render_engine>ogre2</render_engine>
-    </plugin>
   </gazebo>
 </robot>

File: src/bar_examples/magni_description/urdf/inertial.xacro (robot description, xacro)
@@ -1,73 +1,46 @@
-<?xml version="1.0" ?>
-<!--
-Copyright 2019 Osnabruck University, Knowledge Based Systems Group
-https://github.com/uos/uos_tools/tree/kinetic/uos_common_urdf
-Redistribution and use in source and binary forms, with or without modification,
-are permitted provided that the following conditions are met:
-1. Redistributions of source code must retain the above copyright notice,
-   this list of conditions and the following disclaimer.
-2. Redistributions in binary form must reproduce the above copyright notice,
-   this list of conditions and the following disclaimer in the documentation
-   and/or other materials provided with the distribution.
-3. Neither the name of the copyright holder nor the names of its contributors
-   may be used to endorse or promote products derived from this software without
-   specific prior written permission.
-THIS SOFTWARE IS PROVIDED BY THE COPYRIGHT HOLDERS AND CONTRIBUTORS "AS IS"
-AND ANY EXPRESS OR IMPLIED WARRANTIES, INCLUDING, BUT NOT LIMITED TO, THE IMPLIED
-WARRANTIES OF MERCHANTABILITY AND FITNESS FOR A PARTICULAR PURPOSE ARE DISCLAIMED.
-IN NO EVENT SHALL THE COPYRIGHT HOLDER OR CONTRIBUTORS BE LIABLE FOR ANY DIRECT,
-INDIRECT, INCIDENTAL, SPECIAL, EXEMPLARY, OR CONSEQUENTIAL DAMAGES (INCLUDING,
-BUT NOT LIMITED TO, PROCUREMENT OF SUBSTITUTE GOODS OR SERVICES; LOSS OF USE, DATA,
-OR PROFITS; OR BUSINESS INTERRUPTION) HOWEVER CAUSED AND ON ANY THEORY OF LIABILITY,
-WHETHER IN CONTRACT, STRICT LIABILITY, OR TORT (INCLUDING NEGLIGENCE OR OTHERWISE)
-ARISING IN ANY WAY OUT OF THE USE OF THIS SOFTWARE, EVEN IF ADVISED OF THE POSSIBILITY
-OF SUCH DAMAGE.
--->
-<robot xmlns:xacro="http://wiki.ros.org/xacro">
-    <xacro:property name="M_PI" value="3.1415926535897931" />
-    <!-- see https://secure.wikimedia.org/wikipedia/en/wiki/List_of_moment_of_inertia_tensors -->
-    <!-- #################### versions without origin #################### -->
+<xacro:unless value="false"
+    xmlns:xacro="http://www.ros.org/wiki/xacro">    <!-- Wrapper for namespace -->
+    <xacro:property name="M_PI_inertial" value="3.1415926535897931"/>
     <xacro:macro name="sphere_inertial" params="radius mass">
         <inertial>
-            <mass value="${mass}" />
-            <origin xyz="0 0 0" />
-            <inertia ixx="${0.4 * mass * radius * radius}" ixy="0.0" ixz="0.0" iyy="${0.4 * mass * radius * radius}" iyz="0.0" izz="${0.4 * mass * radius * radius}" />
+            <mass value="${mass}"/>
+            <origin xyz="0 0 0"/>
+            <inertia ixx="${0.4 * mass * radius * radius}" ixy="0.0" ixz="0.0" iyy="${0.4 * mass * radius * radius}" iyz="0.0" izz="${0.4 * mass * radius * radius}"/>
         </inertial>
     </xacro:macro>
     <xacro:macro name="cylinder_inertial" params="radius length mass">
         <inertial>
-            <mass value="${mass}" />
-            <origin xyz="0 0 0" />
-            <inertia ixx="${0.0833333 * mass * (3 * radius * radius + length * length)}" ixy="0.0" ixz="0.0" iyy="${0.0833333 * mass * (3 * radius * radius + length * length)}" iyz="0.0" izz="${0.5 * mass * radius * radius}" />
+            <mass value="${mass}"/>
+            <origin xyz="0 0 0"/>
+            <inertia ixx="${0.0833333 * mass * (3 * radius * radius + length * length)}" ixy="0.0" ixz="0.0" iyy="${0.0833333 * mass * (3 * radius * radius + length * length)}" iyz="0.0" izz="${0.5 * mass * radius * radius}"/>
         </inertial>
     </xacro:macro>
     <xacro:macro name="box_inertial" params="x y z mass">
         <inertial>
-            <mass value="${mass}" />
-            <origin xyz="-0.15 0 0.03" />
-            <inertia ixx="${0.0833333 * mass * (y*y + z*z)}" ixy="0.0" ixz="0.0" iyy="${0.0833333 * mass * (x*x + z*z)}" iyz="0.0" izz="${0.0833333 * mass * (x*x + y*y)}" />
+            <mass value="${mass}"/>
+            <origin xyz="-0.15 0 0.03"/>
+            <inertia ixx="${0.0833333 * mass * (y*y + z*z)}" ixy="0.0" ixz="0.0" iyy="${0.0833333 * mass * (x*x + z*z)}" iyz="0.0" izz="${0.0833333 * mass * (x*x + y*y)}"/>
         </inertial>
     </xacro:macro>
-    <!-- #################### versions with origin #################### -->
     <xacro:macro name="sphere_inertial_with_origin" params="radius mass *origin">
         <inertial>
-            <mass value="${mass}" />
-            <xacro:insert_block name="origin" />
-            <inertia ixx="${0.4 * mass * radius * radius}" ixy="0.0" ixz="0.0" iyy="${0.4 * mass * radius * radius}" iyz="0.0" izz="${0.4 * mass * radius * radius}" />
+            <mass value="${mass}"/>
+            <xacro:insert_block name="origin"/>
+            <inertia ixx="${0.4 * mass * radius * radius}" ixy="0.0" ixz="0.0" iyy="${0.4 * mass * radius * radius}" iyz="0.0" izz="${0.4 * mass * radius * radius}"/>
         </inertial>
     </xacro:macro>
     <xacro:macro name="cylinder_inertial_with_origin" params="radius length mass *origin">
         <inertial>
-            <mass value="${mass}" />
-            <xacro:insert_block name="origin" />
-            <inertia ixx="${0.0833333 * mass * (3 * radius * radius + length * length)}" ixy="0.0" ixz="0.0" iyy="${0.0833333 * mass * (3 * radius * radius + length * length)}" iyz="0.0" izz="${0.5 * mass * radius * radius}" />
+            <mass value="${mass}"/>
+            <xacro:insert_block name="origin"/>
+            <inertia ixx="${0.0833333 * mass * (3 * radius * radius + length * length)}" ixy="0.0" ixz="0.0" iyy="${0.0833333 * mass * (3 * radius * radius + length * length)}" iyz="0.0" izz="${0.5 * mass * radius * radius}"/>
         </inertial>
     </xacro:macro>
     <xacro:macro name="box_inertial_with_origin" params="x y z mass *origin">
         <inertial>
-            <mass value="${mass}" />
-            <xacro:insert_block name="origin" />
-            <inertia ixx="${0.0833333 * mass * (y*y + z*z)}" ixy="0.0" ixz="0.0" iyy="${0.0833333 * mass * (x*x + z*z)}" iyz="0.0" izz="${0.0833333 * mass * (x*x + y*y)}" />
+            <mass value="${mass}"/>
+            <xacro:insert_block name="origin"/>
+            <inertia ixx="${0.0833333 * mass * (y*y + z*z)}" ixy="0.0" ixz="0.0" iyy="${0.0833333 * mass * (x*x + z*z)}" iyz="0.0" izz="${0.0833333 * mass * (x*x + y*y)}"/>
         </inertial>
     </xacro:macro>
-</robot>
+</xacro:unless>

File: src/bar_examples/magni_description/urdf/magni.urdf.xacro (robot description, xacro)
@@ -1,8 +1,52 @@
-<?xml version="1.0" encoding='UTF-8'?>
-<robot xmlns:xacro="http://www.ros.org/wiki/xacro">
-  <xacro:property name="wheel_r" value="0.1" />
-  <xacro:property name="wheel_xpos" value="0.11" />
-  <xacro:include filename="$(find magni_description)/urdf/inertial.xacro" />
-  <xacro:macro name="low_friction">
+<xacro:macro name="magni_robot_base_definition"
+  xmlns:xacro="http://www.ros.org/wiki/xacro">
+  <xacro:property name="wheel_r_magni" value="0.1" />
+  <xacro:property name="wheel_xpos_magni" value="0.11" />
+  <!-- START of pasted content that WAS in inertial.xacro -->
+  <xacro:property name="M_PI_inertial" value="3.1415926535897931"/>
+  <xacro:macro name="sphere_inertial" params="radius mass">
+    <inertial>
+      <mass value="${mass}"/>
+      <origin xyz="0 0 0"/>
+      <inertia ixx="${0.4 * mass * radius * radius}" ixy="0.0" ixz="0.0" iyy="${0.4 * mass * radius * radius}" iyz="0.0" izz="${0.4 * mass * radius * radius}"/>
+    </inertial>
+  </xacro:macro>
+  <xacro:macro name="cylinder_inertial" params="radius length mass">
+    <inertial>
+      <mass value="${mass}"/>
+      <origin xyz="0 0 0"/>
+      <inertia ixx="${0.0833333 * mass * (3 * radius * radius + length * length)}" ixy="0.0" ixz="0.0" iyy="${0.0833333 * mass * (3 * radius * radius + length * length)}" iyz="0.0" izz="${0.5 * mass * radius * radius}"/>
+    </inertial>
+  </xacro:macro>
+  <xacro:macro name="box_inertial" params="x y z mass">
+    <inertial>
+      <mass value="${mass}"/>
+      <origin xyz="-0.15 0 0.03"/>
+      <inertia ixx="${0.0833333 * mass * (y*y + z*z)}" ixy="0.0" ixz="0.0" iyy="${0.0833333 * mass * (x*x + z*z)}" iyz="0.0" izz="${0.0833333 * mass * (x*x + y*y)}"/>
+    </inertial>
+  </xacro:macro>
+  <xacro:macro name="sphere_inertial_with_origin" params="radius mass *origin">
+    <inertial>
+      <mass value="${mass}"/>
+      <xacro:insert_block name="origin"/>
+      <inertia ixx="${0.4 * mass * radius * radius}" ixy="0.0" ixz="0.0" iyy="${0.4 * mass * radius * radius}" iyz="0.0" izz="${0.4 * mass * radius * radius}"/>
+    </inertial>
+  </xacro:macro>
+  <xacro:macro name="cylinder_inertial_with_origin" params="radius length mass *origin">
+    <inertial>
+      <mass value="${mass}"/>
+      <xacro:insert_block name="origin"/>
+      <inertia ixx="${0.0833333 * mass * (3 * radius * radius + length * length)}" ixy="0.0" ixz="0.0" iyy="${0.0833333 * mass * (3 * radius * radius + length * length)}" iyz="0.0" izz="${0.5 * mass * radius * radius}"/>
+    </inertial>
+  </xacro:macro>
+  <xacro:macro name="box_inertial_with_origin" params="x y z mass *origin">
+    <inertial>
+      <mass value="${mass}"/>
+      <xacro:insert_block name="origin"/>
+      <inertia ixx="${0.0833333 * mass * (y*y + z*z)}" ixy="0.0" ixz="0.0" iyy="${0.0833333 * mass * (x*x + z*z)}" iyz="0.0" izz="${0.0833333 * mass * (x*x + y*y)}"/>
+    </inertial>
+  </xacro:macro>
+  <!-- END of pasted content from inertial.xacro -->
+  <xacro:macro name="low_friction_magni_internal">
     <collision>
       <surface>
@@ -19,5 +63,5 @@
     </collision>
   </xacro:macro>
-  <xacro:macro name="high_friction">
+  <xacro:macro name="high_friction_magni_internal">
     <collision>
       <surface>
@@ -35,21 +79,14 @@
     </collision>
   </xacro:macro>
-  <link name="base_footprint"/>
-  <joint name="base_footprint_joint" type="fixed">
-    <parent link="base_footprint"/>
-    <child link="base_link"/>
-    <origin xyz="0 0 ${wheel_r}" rpy="0 0 0"/>
-  </joint>
-  <!-- Base Link -->
   <link name="base_link">
-    <origin xyz="-0.25 0 ${0.03}" rpy="0 0 0" />
     <visual>
-      <origin xyz="${-wheel_xpos} 0 ${-wheel_r+0.071}" rpy="0 0 0" />
+      <origin xyz="${-wheel_xpos_magni} 0 ${-wheel_r_magni+0.071}" rpy="0 0 0" />
       <geometry>
-        <mesh filename="file://$(find magni_description)/meshes/magni_body.dae" />
+        <mesh filename="package://magni_description/meshes/magni_body.dae" />
       </geometry>
+      <material name="magni_grey_material"/>
     </visual>
     <collision>
-      <origin xyz="${-wheel_xpos} 0 ${-wheel_r+0.151}" rpy="0 0 0" />
+      <origin xyz="${-wheel_xpos_magni} 0 ${-wheel_r_magni+0.151}" rpy="0 0 0" />
       <geometry>
         <box size="0.398 0.268 0.160"/>
@@ -57,5 +94,5 @@
     </collision>
     <collision>
-      <origin xyz="${-wheel_xpos-0.026} 0 ${-wheel_r+0.248}" rpy="0 0 0" />
+      <origin xyz="${-wheel_xpos_magni-0.026} 0 ${-wheel_r_magni+0.248}" rpy="0 0 0" />
       <geometry>
         <box size="0.375 0.268 0.034"/>
@@ -63,5 +100,5 @@
     </collision>
     <collision>
-      <origin xyz="${-wheel_xpos-0.169} 0.169 ${-wheel_r+0.106}" rpy="0 0 0" />
+      <origin xyz="${-wheel_xpos_magni-0.169} 0.169 ${-wheel_r_magni+0.106}" rpy="0 0 0" />
       <geometry>
         <box size="0.1 0.07 0.07"/>
@@ -69,5 +106,5 @@
     </collision>
     <collision>
-      <origin xyz="${-wheel_xpos-0.169} -0.169 ${-wheel_r+0.106}" rpy="0 0 0" />
+      <origin xyz="${-wheel_xpos_magni-0.169} -0.169 ${-wheel_r_magni+0.106}" rpy="0 0 0" />
       <geometry>
         <box size="0.1 0.07 0.07"/>
@@ -79,23 +116,23 @@
   </link>
   <gazebo reference="base_link">
-    <xacro:low_friction/>
+    <xacro:low_friction_magni_internal/>
   </gazebo>
-  <!-- Macro for defining wheels -->
-  <xacro:macro name="wheel" params="prefix reflect">
-    <link name="${prefix}_wheel">
+  <xacro:macro name="magni_wheel_internal" params="prefix reflect">
+    <link name="${prefix}_wheel_link">
       <collision>
-        <origin xyz="${0.033*reflect} 0 0" rpy="0 ${pi/2} 0" />
+        <origin xyz="${0.033*reflect} 0 0" rpy="0 ${M_PI_inertial/2} 0" />
         <geometry>
-          <cylinder radius="${wheel_r}" length="0.01"/>
+          <cylinder radius="${wheel_r_magni}" length="0.01"/>
         </geometry>
       </collision>
       <visual>
-        <origin xyz="${-0.071*reflect} 0 0" rpy="0 ${(reflect-1)*pi/2} 0" />
+        <origin xyz="${-0.071*reflect} 0 0" rpy="0 ${(reflect-1)*M_PI_inertial/2} 0" />
         <geometry>
-          <mesh filename="file://$(find magni_description)/meshes/front_wheel.dae" />
+          <mesh filename="package://magni_description/meshes/front_wheel.dae" />
         </geometry>
+        <material name="magni_black_material"/>
       </visual>
-      <xacro:cylinder_inertial_with_origin radius="${wheel_r}" length="0.05" mass="1.34">
-        <origin xyz="0 0 0" rpy="0 ${pi/2} 0" />
+      <xacro:cylinder_inertial_with_origin radius="${wheel_r_magni}" length="0.05" mass="1.34">
+        <origin xyz="0 0 0" rpy="0 ${M_PI_inertial/2} 0" />
       </xacro:cylinder_inertial_with_origin>
     </link>
@@ -103,22 +140,19 @@
       <axis xyz="1 0 0" rpy="0 0 0" />
       <parent link="base_link"/>
-      <child link="${prefix}_wheel"/>
-      <origin xyz="0 ${0.163*reflect} 0" rpy="0 0 ${pi/2}"/>
+      <child link="${prefix}_wheel_link"/>
+      <origin xyz="0 ${0.163*reflect} 0" rpy="0 0 ${M_PI_inertial/2}"/>
       <dynamics damping="0.2" friction="0.8"/>
       <limit effort="1000" velocity="10"/>
     </joint>
-    <gazebo reference="${prefix}_wheel">
-      <xacro:high_friction/>
+    <gazebo reference="${prefix}_wheel_link">
+      <xacro:high_friction_magni_internal/>
     </gazebo>
   </xacro:macro>
-  <!--- create wheels -->
-  <xacro:wheel prefix="left" reflect="1"/>
-  <xacro:wheel prefix="right" reflect="-1"/>
-  <!-- Macro for defining caster wheels -->
-  <xacro:macro name="caster_wheel" params="prefix reflect">
-    <link name="${prefix}_caster_wheel">
-      <origin xyz="-0.37 ${reflect*0.169} ${-wheel_r+0.04}" rpy="0 0 0" />
+  <xacro:magni_wheel_internal prefix="left" reflect="1"/>
+  <xacro:magni_wheel_internal prefix="right" reflect="-1"/>
+  <xacro:macro name="magni_caster_wheel_internal" params="prefix reflect">
+    <link name="${prefix}_caster_wheel_link">
       <collision>
-        <origin xyz="-0.27 ${reflect*0.169} ${-wheel_r+0.04}" rpy="0 0 0" />
+        <origin xyz="${-0.27 + (0.37 - 0.27)} ${reflect*0.169} ${-wheel_r_magni+0.04}" rpy="0 0 0" />
         <geometry>
           <sphere radius="0.04"/>
@@ -126,20 +160,32 @@
       </collision>
       <visual>
-        <origin xyz="-0.25 ${reflect*0.169} 0" rpy="0 0 ${pi}" />
+        <origin xyz="${-0.25 + (0.37 - 0.25)} ${reflect*0.169} 0" rpy="0 0 ${M_PI_inertial}" />
         <geometry>
-          <mesh filename="file://$(find magni_description)/meshes/caster_wheel.dae" />
+          <mesh filename="package://magni_description/meshes/caster_wheel.dae" />
         </geometry>
+        <material name="magni_black_material"/>
       </visual>
+      <inertial>
+        <mass value="0.1"/>
+        <origin xyz="0 0 0"/>
+        <inertia ixx="0.001" ixy="0" ixz="0" iyy="0.001" iyz="0" izz="0.001"/>
+      </inertial>
     </link>
     <joint name="${prefix}_caster_wheel_joint" type="fixed">
       <parent link="base_link"/>
-      <child link="${prefix}_caster_wheel"/>
+      <child link="${prefix}_caster_wheel_link"/>
+      <origin xyz="-0.37 ${reflect*0.169} ${-wheel_r_magni+0.04}" rpy="0 0 0" />
     </joint>
-    <gazebo reference="${prefix}_caster_wheel">
-      <xacro:low_friction/>
+    <gazebo reference="${prefix}_caster_wheel_link">
+      <xacro:low_friction_magni_internal/>
     </gazebo>
   </xacro:macro>
-  <!-- and caster wheels )-->
-  <xacro:caster_wheel prefix="left" reflect="1"/>
-  <xacro:caster_wheel prefix="right" reflect="-1"/>
-</robot>
+  <xacro:magni_caster_wheel_internal prefix="left" reflect="1"/>
+  <xacro:magni_caster_wheel_internal prefix="right" reflect="-1"/>
+  <material name="magni_grey_material">
+    <color rgba="0.6 0.6 0.6 1.0"/>
+  </material>
+  <material name="magni_black_material">
+    <color rgba="0.1 0.1 0.1 1.0"/>
+  </material>
+</xacro:macro>
