Commit message: try to accelerate using gpu

File: src/bar_examples/sensors/lidar_2d/lidar_2d.urdf.xacro (robot description, xacro)
@@ -1,42 +1,50 @@
-<robot name="sensor_d435"
-    xmlns:xacro="http://ros.org/wiki/xacro">
+<xacro:unless value="false"
+    xmlns:xacro="http://www.ros.org/wiki/xacro">    <!-- Wrapper for namespace -->
+    <material name="lidar_material_urdf">        <!-- Corrected from xacro:material -->
+        <color rgba="0.3 0.3 0.7 1.0"/>
+    </material>
     <xacro:macro name="lidar_2d" params="world_link_name *origin">
         <link name="lidar_2d_link">
-            <xacro:box_inertial x="0.05" y="0.5" z="0.03" mass="0.13"/>
+            <visual>
+                <origin rpy="0 0 1.5707" xyz="0 0 0"/>
+                <geometry>
+                    <mesh filename="package://sensors/lidar_2d/meshes/lidar_2d_v1.dae"/>
+                </geometry>
+                <material name="lidar_material_urdf"/>
+            </visual>
             <collision name="collision_base">
-                <pose>0 0 0.0175015175 0 0 0</pose>
+                <pose xyz="0 0 0.0175015175" rpy="0 0 0"/>
                 <geometry>
-                    <box size="0.05001062 0.05001062 0.035003035" />
+                    <box size="0.05001062 0.05001062 0.035003035"/>
                 </geometry>
             </collision>
             <collision name="collision_top">
-                <pose>0 0 0.0525045525 0 0 0</pose>
+                <pose xyz="0 0 0.0525045525" rpy="0 0 0"/>
                 <geometry>
                     <cylinder radius="0.02" length="0.035003035"/>
                 </geometry>
             </collision>
-            <visual name="visual">
-                <pose>0 0 0 0 0 1.5707</pose>
-                <geometry>
-                    <mesh filename="package://sensors/lidar_2d/meshes/lidar_2d_v1.dae" />
-                </geometry>
-            </visual>
+            <inertial>
+                <mass value="0.1"/>
+                <origin xyz="0 0 0.025" rpy="0 0 0"/>
+                <inertia ixx="0.0001" ixy="0" ixz="0" iyy="0.0001" iyz="0" izz="0.0001"/>
+            </inertial>
         </link>
         <gazebo reference="lidar_2d_link">
             <sensor name="lidar_2d_v1" type="gpu_ray">
-                <topic>lidar</topic>
-                <pose>0 0 0.0525045525 0 0 0</pose>
+                <topic>/gz/krytn_lidar/scan</topic>
+                <pose xyz="0 0 0.0525045525" rpy="0 0 0"/>
                 <ray>
                     <scan>
                         <horizontal>
-                            <samples>180</samples>
+                            <samples>360</samples>
                             <resolution>1</resolution>
-                            <min_angle>-2.356195</min_angle>
-                            <max_angle>2.356195</max_angle>
+                            <min_angle>-3.14159</min_angle>
+                            <max_angle>3.14159</max_angle>
                         </horizontal>
                     </scan>
                     <range>
-                        <min>0.060</min>
-                        <max>5</max>
+                        <min>0.10</min>
+                        <max>10.0</max>
                         <resolution>0.01</resolution>
                     </range>
@@ -44,17 +52,17 @@
                         <type>gaussian</type>
                         <mean>0.0</mean>
-                        <stddev>0.001</stddev>
+                        <stddev>0.01</stddev>
                     </noise>
                 </ray>
-                <always_on>0</always_on>
+                <always_on>true</always_on>
                 <update_rate>10</update_rate>
-                <visualize>false</visualize>
+                <visualize>true</visualize>
             </sensor>
         </gazebo>
         <joint name="lidar_2d_joint" type="fixed">
-            <child link="lidar_2d_link" />
-            <parent link="${world_link_name}" />
+            <parent link="${world_link_name}"/>
+            <child link="lidar_2d_link"/>
             <xacro:insert_block name="origin"/>
         </joint>
     </xacro:macro>
-</robot>
+</xacro:unless>

File: src/bar_examples/sensors/realsense_d435/realsense.urdf.xacro (robot description, xacro)
@@ -1,18 +1,15 @@
-<robot name="sensor_d435"
-    xmlns:xacro="http://ros.org/wiki/xacro">
+<xacro:unless value="false"
+    xmlns:xacro="http://www.ros.org/wiki/xacro">    <!-- Wrapper for namespace -->
     <xacro:macro name="realsense" params="world_link_name *origin">
+        <material name="realsense_material_urdf">            <!-- DEFINED INSIDE MACRO -->
+            <color rgba="0.5 0.5 0.6 1.0"/>
+        </material>
         <link name="realsense_link">
-            <xacro:box_inertial x="0.02" y="0.1" z="0.01" mass="0.06"/>
-            <collision name="collision">
-                <origin rpy="0 0 ${pi/2}"/>
-                <geometry>
-                    <mesh filename="package://sensors/realsense_d435/meshes/realsense.dae" />
-                </geometry>
-            </collision>
-            <visual name= "visual">
-                <origin rpy="0 0 ${pi/2}"/>
+            <visual>
+                <origin rpy="0 0 1.5707963267948966"/>
                 <geometry>
                     <mesh filename="package://sensors/realsense_d435/meshes/realsense.dae"/>
                 </geometry>
+                <material name="realsense_material_urdf"/>
                 <gazebo>
                     <material>
@@ -27,5 +24,4 @@
                             </metal>
                         </pbr>
-                        <!-- fallback to script if no PBR support-->
                         <script>
                             <uri>package://sensors/realsense_d435/materials/scripts/</uri>
@@ -36,11 +32,18 @@
                 </gazebo>
             </visual>
+            <collision>
+                <origin rpy="0 0 1.5707963267948966"/>
+                <geometry>
+                    <mesh filename="package://sensors/realsense_d435/meshes/realsense.dae"/>
+                </geometry>
+            </collision>
+            <xacro:box_inertial x="0.02" y="0.1" z="0.01" mass="0.06"/>
         </link>
         <gazebo reference="realsense_link">
-            <sensor name="realsense_d435" type="rgbd_camera">
+            <sensor name="realsense_d435_sensor" type="rgbd_camera">
                 <update_rate>10</update_rate>
-                <topic>realsense</topic>
-                <camera name="camera">
-                    <optical_frame_id>realsense_link</optical_frame_id>
+                <topic>/gz/krytn_realsense</topic>
+                <camera name="rs_camera">
+                    <optical_frame_id>realsense_depth_optical_frame</optical_frame_id>
                     <horizontal_fov>1.0472</horizontal_fov>
                     <image>
@@ -50,15 +53,29 @@
                     </image>
                     <clip>
-                        <near>0.01</near>
-                        <far>300</far>
+                        <near>0.1</near>
+                        <far>10.0</far>
                     </clip>
+                    <depth_camera/>
+                    <noise>
+                        <type>gaussian</type>
+                        <mean>0.0</mean>
+                        <stddev>0.007</stddev>
+                    </noise>
                 </camera>
+                <always_on>true</always_on>
+                <visualize>true</visualize>
             </sensor>
         </gazebo>
+        <joint name="realsense_depth_joint" type="fixed">
+            <origin rpy="-1.57079632679 0 -1.57079632679" xyz="0 0 0"/>
+            <parent link="realsense_link"/>
+            <child link="realsense_depth_optical_frame"/>
+        </joint>
+        <link name="realsense_depth_optical_frame"/>
         <joint name="realsense_joint" type="fixed">
-            <child link="realsense_link" />
-            <parent link="${world_link_name}" />
+            <parent link="${world_link_name}"/>
+            <child link="realsense_link"/>
             <xacro:insert_block name="origin"/>
         </joint>
     </xacro:macro>
-</robot>
+</xacro:unless>
